Commit message: Updated the rotations of the joint

File: urdf/fanuc.urdf (robot description, URDF)
Before this commit: robot fanuc, 7 links, 6 joints
Joints:
- joint link_2_to_link_3: axis (none) -> 1 0.0 0.0; limit (none) -> lower=0 upper=3.14 effort=0.0 velocity=0.0; origin xyz=0.0 0.0 1.1 rpy=3.14 0.0 -1.57 -> xyz=0.0 0.0 0.95 rpy=3.14 0.0 -1.57; type fixed -> revolute
- joint link_3_to_link_4: origin xyz=-0.06 -1. 0.0 rpy=0.0 3.14 -1.57 -> xyz=-0.06 -1.2 0.0 rpy=0.0 3.14 -1.57
- joint link_4_to_link_5: origin xyz=0.12 0.0 0.0 rpy=0.0 0.0 1.57 -> xyz=0.12 0.0 0.0 rpy=0.0 0.0 3.14
- joint link_5_to_link_6: origin xyz=0.17 0.0 0.0 rpy=0.0 0.0 0.0 -> xyz=0.18 0.0 0.0 rpy=0.0 0.0 0.0
